File: kicad/RGBStacks.kicad_pcb (KiCad board)
At the start: 2 copper layers, 68.6 x 50.2 mm, 27 parts, among them J1 RJ45_8, J2 CONN_01X06, J3 CONN_02X12, J4 CONN_02X04, U1 PIC12F1572, U2 PIC12F1572, U3 PIC12F1572, U4 PIC12F1572, U5 ULN2003A, U6 ULN2003A

Commit message: Update PCB designs.
Parts:
- added C1: CP1, Capacitors_SMD:C_0805_HandSoldering, B.Cu at (141.0, 92.7)
- added C2: CP1, Capacitors_SMD:C_0805_HandSoldering, B.Cu at (141.0, 116.8)
- added C3: CP1, Capacitors_SMD:C_0805_HandSoldering, B.Cu at (141.0, 104.8)
- added C4: CP1, Capacitors_SMD:C_0805_HandSoldering, B.Cu at (141.0, 80.6)
Routing:
- net GND: track 147.1 -> 168.4 mm, vias 0 -> 1
- net +5V: track 155.3 -> 165.3 mm

Commit message: PCB tweaks.
Other:
- board text added: "0.1uF"
Changed lines of the file:
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@@
     (area 115.294999 73.447 191.088334 124.011)
     (thickness 1.6)
-    (drawings 58)
+    (drawings 62)
     (tracks 211)
     (zones 0)
@@
     (uvia_dia 0.3)
     (uvia_drill 0.1)
+    (add_net GND)
     (add_net MCLR1)
     (add_net MCLR2)
@@
     (uvia_dia 0.3)
     (uvia_drill 0.1)
-    (add_net GND)
   )
   (module Connectors:1pin (layer F.Cu)
@@
       (effects (font (size 1 1) (thickness 0.15)))
     )
-    (fp_text value PIC12F1572 (at 4.445 4.064 180) (layer F.Fab)
+    (fp_text value PIC12F1572 (at 3.81 4.064 180) (layer F.Fab)
       (effects (font (size 1 1) (thickness 0.15)))
     )
@@
     )
   )
+  (gr_text 0.1uF (at 142.494 116.84 90) (layer B.SilkS)
+    (effects (font (size 0.5 0.5) (thickness 0.1)) (justify mirror))
+  )
+  (gr_text 0.1uF (at 142.494 104.775 90) (layer B.SilkS)
+    (effects (font (size 0.5 0.5) (thickness 0.1)) (justify mirror))
+  )
+  (gr_text 0.1uF (at 142.494 92.71 90) (layer B.SilkS)
+    (effects (font (size 0.5 0.5) (thickness 0.1)) (justify mirror))
+  )
+  (gr_text 0.1uF (at 142.494 80.772 90) (layer B.SilkS)
+    (effects (font (size 0.5 0.5) (thickness 0.1)) (justify mirror))
+  )
   (gr_text 8-9.7 (at 168.529 104.902) (layer F.SilkS)
     (effects (font (size 0.5 0.5) (thickness 0.1)))
@@
   (segment (start 126.238 93.091) (end 129.794 89.535) (width 0.5) (layer B.Cu) (net 1))
   (segment (start 126.238 98.552) (end 126.238 93.091) (width 0.5) (layer B.Cu) (net 1))
-  (segment (start 175.514 106.045) (end 175.514 118.745) (width 0.5) (layer B.Cu) (net 1) (status 400000))
+  (segment (start 175.514 106.045) (end 175.514 118.745) (width 0.5) (layer B.Cu) (net 1))
   (segment (start 142.748 122.428) (end 140.97 120.65) (width 0.5) (layer B.Cu) (net 1))
   (segment (start 172.72 122.428) (end 142.748 122.428) (width 0.5) (layer B.Cu) (net 1))
@@
   (segment (start 139.065 112.395) (end 139.065 118.745) (width 0.5) (layer B.Cu) (net 1))
   (segment (start 140.97 110.49) (end 139.065 112.395) (width 0.5) (layer B.Cu) (net 1))
+  (segment (start 140.97 88.9) (end 142.24 87.757) (width 0.25) (layer B.Cu) (net 2))
+  (segment (start 142.24 77.978) (end 140.97 76.835) (width 0.25) (layer B.Cu) (net 2))
+  (segment (start 142.24 87.757) (end 142.24 77.978) (width 0.25) (layer B.Cu) (net 2))
   (segment (start 120.65 106.68) (end 129.286 115.316) (width 0.5) (layer B.Cu) (net 2))
   (via (at 129.286 115.316) (size 0.6) (drill 0.4) (layers F.Cu B.Cu) (net 2))
@@
   (segment (start 140.97 115.59) (end 140.97 113.03) (width 0.5) (layer B.Cu) (net 2))
   (segment (start 140.97 76.835) (end 135.128 82.677) (width 0.5) (layer B.Cu) (net 2))
+  (segment (start 135.128 82.677) (end 135.128 85.471) (width 0.5) (layer B.Cu) (net 2))
   (segment (start 135.128 85.471) (end 132.334 88.265) (width 0.5) (layer B.Cu) (net 2))
-  (segment (start 135.128 82.677) (end 135.128 85.471) (width 0.5) (layer B.Cu) (net 2))
   (segment (start 120.65 106.68) (end 118.618 104.648) (width 0.5) (layer B.Cu) (net 2))
   (segment (start 124.46 86.995) (end 129.794 86.995) (width 0.5) (layer B.Cu) (net 2))
@@
   (segment (start 153.67 95.885) (end 153.797 95.885) (width 0.5) (layer B.Cu) (net 2))
   (segment (start 153.797 95.885) (end 155.321 94.361) (width 0.5) (layer B.Cu) (net 2))
+  (segment (start 155.321 94.361) (end 155.321 77.089) (width 0.5) (layer B.Cu) (net 2))
+  (segment (start 155.321 77.089) (end 153.543 75.311) (width 0.5) (layer B.Cu) (net 2))
+  (segment (start 153.543 75.311) (end 142.494 75.311) (width 0.5) (layer B.Cu) (net 2))
   (segment (start 142.494 75.311) (end 140.97 76.835) (width 0.5) (layer B.Cu) (net 2))
-  (segment (start 153.543 75.311) (end 142.494 75.311) (width 0.5) (layer B.Cu) (net 2))
-  (segment (start 155.321 77.089) (end 153.543 75.311) (width 0.5) (layer B.Cu) (net 2))
-  (segment (start 155.321 94.361) (end 155.321 77.089) (width 0.5) (layer B.Cu) (net 2))
   (segment (start 153.67 119.38) (end 153.797 119.38) (width 0.5) (layer B.Cu) (net 2))
   (segment (start 153.797 119.38) (end 155.321 117.856) (width 0.5) (layer B.Cu) (net 2))
   (segment (start 155.321 117.856) (end 155.321 97.536) (width 0.5) (layer B.Cu) (net 2))
   (segment (start 155.321 97.536) (end 153.67 95.885) (width 0.5) (layer B.Cu) (net 2))
-  (segment (start 140.97 113.03) (end 142.24 111.76) (width 0.5) (layer B.Cu) (net 2))
-  (segment (start 142.24 102.235) (end 140.97 100.965) (width 0.5) (layer B.Cu) (net 2))
-  (segment (start 142.24 111.76) (end 142.24 102.235) (width 0.5) (layer B.Cu) (net 2))
-  (segment (start 140.97 100.965) (end 142.24 99.695) (width 0.5) (layer B.Cu) (net 2))
-  (segment (start 142.24 99.695) (end 142.24 90.17) (width 0.5) (layer B.Cu) (net 2))
-  (segment (start 142.24 90.17) (end 140.97 88.9) (width 0.5) (layer B.Cu) (net 2))
-  (segment (start 140.97 88.9) (end 142.24 87.63) (width 0.5) (layer B.Cu) (net 2))
-  (segment (start 142.24 87.63) (end 142.24 78.105) (width 0.5) (layer B.Cu) (net 2))
-  (segment (start 142.24 78.105) (end 140.97 76.835) (width 0.5) (layer B.Cu) (net 2))
+  (segment (start 140.97 113.03) (end 142.24 111.76) (width 0.25) (layer B.Cu) (net 2))
+  (segment (start 142.24 102.235) (end 140.97 100.965) (width 0.25) (layer B.Cu) (net 2))
+  (segment (start 142.24 111.76) (end 142.24 102.235) (width 0.25) (layer B.Cu) (net 2))
+  (segment (start 140.97 100.965) (end 142.24 99.695) (width 0.25) (layer B.Cu) (net 2))
+  (segment (start 142.24 99.695) (end 142.24 90.17) (width 0.25) (layer B.Cu) (net 2))
+  (segment (start 142.24 90.17) (end 140.97 88.9) (width 0.25) (layer B.Cu) (net 2))
   (segment (start 148.59 84.455) (end 151.511 87.376) (width 0.25) (layer F.Cu) (net 3))
   (segment (start 152.908 115.57) (end 166.116 115.57) (width 0.25) (layer F.Cu) (net 3))

Commit message: Updated PCB.
Parts:
- removed 10K, R10, R11, R12, R13, R2, R3, R4, R5, R6, R7, R8, R9: R, Resistors_SMD:R_0603_HandSoldering
- added 10K1: R, Resistors_THT:R_Axial_DIN0207_L6.3mm_D2.5mm_P7.62mm_Horizontal, F.Cu at (180.1, 109.3)
- added 4.3: R, Resistors_THT:R_Axial_DIN0207_L6.3mm_D2.5mm_P7.62mm_Horizontal, F.Cu at (167.5, 83.9)
- added 4.3: R, Resistors_THT:R_Axial_DIN0207_L6.3mm_D2.5mm_P7.62mm_Horizontal, F.Cu at (167.5, 94.6)
- added 4.3: R, Resistors_THT:R_Axial_DIN0207_L6.3mm_D2.5mm_P7.62mm_Horizontal, F.Cu at (167.5, 105.3)
- added 4.7: R, Resistors_THT:R_Axial_DIN0207_L6.3mm_D2.5mm_P7.62mm_Horizontal, F.Cu at (167.5, 87.5)
- added 4.7: R, Resistors_THT:R_Axial_DIN0207_L6.3mm_D2.5mm_P7.62mm_Horizontal, F.Cu at (167.5, 98.2)
- added 4.7: R, Resistors_THT:R_Axial_DIN0207_L6.3mm_D2.5mm_P7.62mm_Horizontal, F.Cu at (167.5, 108.8)
- added 5.6: R, Resistors_THT:R_Axial_DIN0207_L6.3mm_D2.5mm_P7.62mm_Horizontal, F.Cu at (167.5, 112.4)
- added 5.6: R, Resistors_THT:R_Axial_DIN0207_L6.3mm_D2.5mm_P7.62mm_Horizontal, F.Cu at (167.5, 116.0)
- added 5.6: R, Resistors_THT:R_Axial_DIN0207_L6.3mm_D2.5mm_P7.62mm_Horizontal, F.Cu at (167.5, 119.5)
- added 7.5: R, Resistors_THT:R_Axial_DIN0207_L6.3mm_D2.5mm_P7.62mm_Horizontal, F.Cu at (167.5, 80.4)
- added 7.5: R, Resistors_THT:R_Axial_DIN0207_L6.3mm_D2.5mm_P7.62mm_Horizontal, F.Cu at (167.5, 91.1)
- added 7.5: R, Resistors_THT:R_Axial_DIN0207_L6.3mm_D2.5mm_P7.62mm_Horizontal, F.Cu at (167.5, 101.7)
- moved J2 16.1 mm to (115.6, 116.8), turned to 90 degrees
- moved C1 6.21 mm to (135.6, 95.9)
- moved U3 6.21 mm to (135.6, 111.8)
- moved C2 6.21 mm to (135.6, 120.0)
- moved C3 6.21 mm to (135.6, 108.0)
- moved C4 6.21 mm to (135.6, 83.8)
- moved U1 6.21 mm to (135.6, 87.6)
- moved U2 6.21 mm to (135.6, 99.7)
- moved U4 6.21 mm to (135.6, 123.8)
- moved U6 6.21 mm to (148.3, 104.8)
- moved U5 6.21 mm to (148.3, 81.3)
- moved J4 4.88 mm to (172.6, 116.0)
- moved REF** 4.77 mm to (116.1, 123.3)
- moved REF** 4.68 mm to (116.0, 80.5)
- moved J1 4.58 mm to (120.1, 92.1)
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Routing:
- net RX/PGC: track 87.4 -> 74.7 mm
- net +5V: track 165.3 -> 176.9 mm
- net MCLR1: track 51.0 -> 61.7 mm
- net GND: track 168.4 -> 179.0 mm, vias 1 -> 0
- net TX/PGD: track 79.7 -> 69.3 mm
- net MCLR2: track 41.4 -> 50.4 mm
- net Net-(J3-Pad23): track 3.47 -> 12.4 mm
- net MCLR4: track 22.2 -> 30.3 mm
- net MCLR3: track 32.2 -> 40.3 mm
- net Net-(J3-Pad21): track 3.47 -> 11.4 mm
- net Net-(J3-Pad19): track 3.47 -> 10.4 mm
- net Net-(R11-Pad2): track 10.8 -> 4.06 mm
- net Net-(R12-Pad2): track 10.8 -> 4.36 mm
- net Net-(R10-Pad2): track 10.7 -> 4.36 mm
- net Net-(R9-Pad2): track 10.7 -> 4.78 mm
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Other:
- board size 68.6 x 50.2 mm -> 71.5 x 50.2 mm
- net class MaxCurrent added: clearance 0.2, trace_width 2.5, via_dia 0.6, via_drill 0.4
- board text added: "1: RX 2: TX 3,4: GND 5,6: 5V"
- board text added: "5"
- board text added: "7"
- board text added: "8"
- board text added: "Revision 2"
- board text removed: "6.3-7.4"
- board text removed: "8-9.7"
- board text removed: "9.1-10.9"
- board text removed: "RX"
- board text removed: "Revision 1"
- board text removed: "TX"
